File: pz-hardware-logic.kicad_pcb (KiCad board)
At the start: 2 copper layers, 0 parts

Commit message: Add IC and some power filters. Started reset network.
Parts:
- added C1: 10uF, Capacitor_THT:CP_Axial_L10.0mm_D4.5mm_P15.00mm_Horizontal, F.Cu at (135.9, 50.8)
- added C2: 1uF, Capacitor_THT:CP_Axial_L10.0mm_D4.5mm_P15.00mm_Horizontal, F.Cu at (111.6, 57.3)
- added J1: Logic Header, Connector_PinHeader_2.54mm:PinHeader_2x15_P2.54mm_Vertical, F.Cu at (105.0, 49.6)
- added R1: 10k, Resistor_THT:R_Axial_DIN0411_L9.9mm_D3.6mm_P20.32mm_Horizontal, F.Cu at (111.8, 49.9)
- added U1: ESP32-WROOM-32U, RF_Module:ESP32-WROOM-32U, F.Cu at (137.2, 77.5)
